File: PCB/PicoprobeTester.kicad_pcb (KiCad board)
At the start: 2 copper layers, 116.7 x 55.7 mm, 10 parts, among them J1 External_Connections

Commit message: Version 2 changes.
Parts:
- SW1: renamed from Connect UART
- SW2: renamed from Reset; footprint Connector_PinHeader_2.54mm:PinHeader_1x02_P2.54mm_Vertical -> ThePCSite:Alps_SKRGAFD010
- moved SW2 1.03 mm to (93.9, 114.6), turned to 0 degrees
- renumbered SWD to J2, PicoProbe to PicoProbe1, Target to Target1
Connections:
- J1 pad 2: GND -> /VBus
- PicoProbe1 pad 40: unconnected-(PicoProbe1-VBUS-Pad40) -> /VBus
- PicoProbe1 pad 41: unconnected-(PicoProbe1-SWCLK-Pad41) -> /SWCLK
- PicoProbe1 pad 43: unconnected-(PicoProbe1-SWDIO-Pad43) -> /SWDIO
- SW2 pad 1: GND -> /TT_Run
- SW2 pad 2: /TT_Run -> GND
- Target1 pad 40: unconnected-(Target1-VBUS-Pad40) -> /VBus
- Target1 pad 41: unconnected-(Target1-SWCLK-Pad41) -> /SWCLK
- Target1 pad 43: unconnected-(Target1-SWDIO-Pad43) -> /SWDIO
Routing:
- net /SWDIO: track 47.1 -> 142.4 mm
- net /VBus: track 0.00 -> 80.8 mm
- net +5V: track 0.00 -> 80.4 mm
- net /SWCLK: track 64.0 -> 125.8 mm
Other:
- board text added: "Pico Debugger v2.0"
- board text added: "Reset"
