File: PCB/PicoprobeTester.kicad_sch (KiCad schematic)
At the start: 10 parts, among them J1 External_Connections, J2 SWD, SW1 UART, SW2 Reset_Target

Commit message: Version 2 changes.
Parts:
- SW2: footprint Connector_PinHeader_2.54mm:PinHeader_1x02_P2.54mm_Vertical -> ThePCSite:Alps_SKRGAFD010
Connections:
- net GND: now also SW2.2; no longer J1.2 (Pin_2), SW2.1
- net SWCLK: now also PicoProbe1.41 (SWCLK), Target1.41 (SWCLK)
- net SWDIO: now also PicoProbe1.43 (SWDIO), Target1.43 (SWDIO)
- net TT_Run: now also SW2.1; no longer SW2.2
- net VBus: now reaches Target1.40 (VBUS)
- net VBus: now also J1.2 (Pin_2), PicoProbe1.40 (VBUS)
- no-connect marks 26 -> 24
Other:
- moved on the sheet: SW2
Changed lines of the file:
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@@
   (no_connect (at 87.63 77.47))
   (no_connect (at 87.63 57.15))
-  (no_connect (at 87.63 41.91))
   (no_connect (at 87.63 74.93))
   (no_connect (at 52.07 87.63))
@@
   (no_connect (at 87.63 64.77))
   (no_connect (at 52.07 41.91))
-  (no_connect (at 162.56 43.18))
   (no_connect (at 52.07 82.55))
   (no_connect (at 52.07 64.77))
@@
     (effects (font (size 1.27 1.27)) (justify right bottom))
   )
+  (label "VBus" (at 210.82 44.45 0) (fields_autoplaced)
+    (effects (font (size 1.27 1.27)) (justify left bottom))
+  )
   (label "GND" (at 198.12 87.63 180) (fields_autoplaced)
     (effects (font (size 1.27 1.27)) (justify right bottom))
@@
     (effects (font (size 1.27 1.27)) (justify left bottom))
   )
+  (label "SWDIO" (at 72.39 95.25 270) (fields_autoplaced)
+    (effects (font (size 1.27 1.27)) (justify right bottom))
+  )
   (label "TT_UART_Rx" (at 198.12 46.99 180) (fields_autoplaced)
     (effects (font (size 1.27 1.27)) (justify right bottom))
@@
     (effects (font (size 1.27 1.27)) (justify right bottom))
   )
+  (label "VBus" (at 162.56 43.18 0) (fields_autoplaced)
+    (effects (font (size 1.27 1.27)) (justify left bottom))
+  )
   (label "GND" (at 198.12 74.93 180) (fields_autoplaced)
     (effects (font (size 1.27 1.27)) (justify right bottom))
@@
     (effects (font (size 1.27 1.27)) (justify left bottom))
   )
+  (label "SWCLK" (at 142.24 96.52 270) (fields_autoplaced)
+    (effects (font (size 1.27 1.27)) (justify right bottom))
+  )
   (label "PP_UART_Tx" (at 256.54 55.88 180) (fields_autoplaced)
     (effects (font (size 1.27 1.27)) (justify right bottom))
@@
     (effects (font (size 1.27 1.27)) (justify left bottom))
   )
+  (label "SWCLK" (at 67.31 95.25 270) (fields_autoplaced)
+    (effects (font (size 1.27 1.27)) (justify right bottom))
+  )
   (label "TT_UART_Tx" (at 127 43.18 180) (fields_autoplaced)
     (effects (font (size 1.27 1.27)) (justify right bottom))
   )
-  (label "GND" (at 210.82 44.45 0) (fields_autoplaced)
+  (label "VBus" (at 87.63 41.91 0) (fields_autoplaced)
     (effects (font (size 1.27 1.27)) (justify left bottom))
   )
@@
     (effects (font (size 1.27 1.27)) (justify left bottom))
   )
+  (label "SWDIO" (at 147.32 96.52 270) (fields_autoplaced)
+    (effects (font (size 1.27 1.27)) (justify right bottom))
+  )
   (label "TT_Run" (at 269.24 82.55 0) (fields_autoplaced)
     (effects (font (size 1.27 1.27)) (justify left bottom))
@@
     (effects (font (size 1.27 1.27)) (justify right bottom))
   )
-  (symbol (lib_id "Switch:SW_Push") (at 264.16 82.55 0) (unit 1)
+  (symbol (lib_id "Switch:SW_Push") (at 264.16 82.55 180) (unit 1)
     (in_bom yes) (on_board yes) (dnp no) (fields_autoplaced)
-    (property "Reference" "SW2" (at 264.16 76.049 0)
+    (property "Reference" "SW2" (at 264.16 77.47 0)
       (effects (font (size 1.27 1.27)))
     )
-    (property "Value" "Reset_Target" (at 264.16 78.097 0)
+    (property "Value" "Reset_Target" (at 264.16 80.01 0)
       (effects (font (size 1.27 1.27)))
     )
-    (property "Footprint" "Connector_PinHeader_2.54mm:PinHeader_1x02_P2.54mm_Vertical" (at 264.16 77.47 0)
+    (property "Footprint" "ThePCSite:Alps_SKRGAFD010" (at 264.16 87.63 0)
       (effects (font (size 1.27 1.27)) hide)
     )
-    (property "Datasheet" "~" (at 264.16 77.47 0)
+    (property "Datasheet" "~" (at 264.16 87.63 0)
       (effects (font (size 1.27 1.27)) hide)
     )
